File: cad/controller/controller.sch (KiCad schematic (older format))
At the start: 14 parts

Commit message: Chose ethernet jack and completed schematic capture for W5500.
Parts:
- removed C? (x4): C, symbol Device:C
- removed L?: L_Core_Ferrite, symbol Device:L_Core_Ferrite
- removed U?: ATmega328-PU, Package_DIP:DIP-28_W7.62mm, symbol MCU_Microchip_ATmega:ATmega328-PU
- removed Y?: Crystal, symbol Device:Crystal
- added C? (x2): 10nF, symbol Device:C
- added C?: 22nF, symbol Device:C
- added C? (x2): 6.8nF, symbol Device:C
- added C? (x2): C, symbol Device:C
- added C? (x2): 18pF, symbol Device:C
- added C?: 4.7uF, symbol Device:C
- added J?: RJ45_jack_POE, symbol custom:RJ45_jack_POE
- added JP? (x2): Jumper, symbol Device:Jumper
- added L?: L_Core_Ferrite, symbol Device:L_Core_Ferrite
- added R? (x5): 0, symbol Device:R
- added R? (x4): 49.9, symbol Device:R
- added R?: 12k4, symbol Device:R
- added R?: 10, symbol Device:R
- added R? (x3): 10k, symbol Device:R
- added R? (x3): DNF, symbol Device:R
- added R? (x2): 330, symbol Device:R
- added R?: 1M, symbol Device:R
- added Y?: Crystal, symbol Device:Crystal
Connections:
- net labels added: 3V3_ANA, ACT_LED, CS, INT, LINK_LED, MISO, MOSI, PIN_12V_JACK, PIN_12V_POE, RST_W5500, SCLK
- net labels removed: AREF
- wire segments 46 -> 187
- no-connect marks 0 -> 5
Other:
- note added: "25 MHz"
- note added: "<1%"
- note added: "ARJM11C7-114-BA-EW2"
- note added: "See http://wizwiki.net/wiki/lib/exe/fetch.php/\nproducts:w5500:w5500_sch_v110_use_mag_.png?cache="
- note added: "VC2 is POE on\nJ4/5 (VC2+) and\nJ7/8 (VC2-)"
- moved on the sheet: C?, U?

Commit message: Finished majority of schematic capture. Need to add sensors and sensor headers
Parts:
- removed R? (x3): DNF, symbol Device:R
- added JP? (x3): Jumper, symbol Device:Jumper
- added R? (x2): 0, symbol Device:R
- added R?: DNF, symbol Device:R
- added R?: 100k, symbol Device:R
- added R?: 4.7k, symbol Device:R
- added SW?: SW_Push, symbol Switch:SW_Push
- added U?: TXB0104D, Package_SO:SOIC-14_3.9x8.7mm_P1.27mm, symbol Logic_LevelTranslator:TXB0104D
- added U?: CAT811STBI-GT3, Package_TO_SOT_SMD:SOT-143, symbol Power_Supervisor:CAT811STBI-GT3
Connections:
- net labels added: CS_5V, INT_W5500, MISO_5V, MOSI_5V, RST, SCLK_5V
- net labels removed: INT
- wire segments 187 -> 228
Other:
- note added: "W5500 RSTn internal\npullup > 62k"
- moved on the sheet: C?, J?, JP?, R?, U?, Y?

Commit message: Added decoupling inductors and capacitors
Parts:
- removed C? (x2): 22uF, Capacitor_SMD:C_0603_1608Metric, symbol Device:CP
- removed C? (x2): 10uF, Capacitor_SMD:C_0603_1608Metric, symbol Device:CP
- removed C? (x2): C, symbol Device:C
- removed L?: L_Core_Ferrite, symbol Device:L_Core_Ferrite
- removed U?: TXB0104D, Package_SO:SOIC-14_3.9x8.7mm_P1.27mm, symbol Logic_LevelTranslator:TXB0104D
- added C? (x8): 100nF, Capacitor_SMD:C_0603_1608Metric, symbol Device:C
- added C? (x6): 10uF, Capacitor_SMD:C_0603_1608Metric, symbol Device:C
- added C?: 33uF, Capacitor_THT:CP_Radial_D4.0mm_P2.00mm, symbol Device:CP
- added FB?: BLM21, Inductor_SMD:L_0805_2012Metric, symbol Device:Ferrite_Bead
- added FB? (x2): BLM21, symbol Device:Ferrite_Bead
- added J?: Barrel_Jack, symbol Connector:Barrel_Jack
- added TP? (x2): TestPoint, symbol Connector:TestPoint
- C? (x8): footprint (none) -> Capacitor_SMD:C_0603_1608Metric
- R? (x22): footprint (none) -> Resistor_SMD:R_0603_1608Metric
- Y?: value Crystal -> 25MHz
Connections:
- net labels removed: CS_5V, MISO_5V, MOSI_5V, SCLK_5V
- wire segments 228 -> 259
Other:
- note added: "25 MHz\nECS-250-18-5PX-F-TR (50ppm)\n"
- note removed: "25 MHz"
- moved on the sheet: C?, JP?, R?, U?

Commit message: Ordered components
Parts:
- added D1: D, symbol Device:D
- gave numbers to parts that had none: 63
Connections:
- net PIN_12V: now also D1.1 (K); no longer JP4.1, JP5.2
- new net: D1.2 (A), JP4.1, JP5.2
Other:
- moved on the sheet: JP4, JP5

Commit message: Added custom libraries submodule and updated the symbol tables in the kicad projects
Parts:
- J1: symbol custom:RJ45_jack_POE -> custom_passive:RJ45_jack_POE
- U4: symbol custom:W5500 -> custom_digital:W5500
Changed lines of the file:
@@
 PIN_12V
 $Comp
-L custom:W5500 U4
+L custom_digital:W5500 U4
 U 1 1 62228853
 P 4750 4150
@@
 <1%
 $Comp
-L custom:RJ45_jack_POE J1
+L custom_passive:RJ45_jack_POE J1
 U 1 1 62344D7E
 P 9600 4950

Commit message: Started associating footprints with controller schematic
Parts:
- D1: footprint (none) -> Diode_THT:D_DO-41_SOD81_P7.62mm_Horizontal
- FB2, FB3: footprint (none) -> Inductor_SMD:L_0805_2012Metric
- J2: footprint (none) -> Connector_BarrelJack:BarrelJack_Horizontal; symbol Connector:Barrel_Jack -> Connector:Barrel_Jack_MountingPin
- JP1, JP2, JP3, JP4, JP5: footprint (none) -> Connector_PinSocket_2.54mm:PinSocket_1x02_P2.54mm_Vertical
- SW1: footprint (none) -> Button_Switch_THT:SW_PUSH_6mm
- TP1, TP2: footprint (none) -> TestPoint:TestPoint_Pad_2.5x2.5mm
- U4: footprint (none) -> Package_QFP:LQFP-48_7x7mm_P0.5mm
- Y1: footprint (none) -> Crystal:Crystal_SMD_HC49-SD_HandSoldering
Changed lines of the file:
@@
 F 0 "U4" H 5644 4196 50  0000 L CNN
 F 1 "W5500" H 5644 4105 50  0000 L CNN
-F 2 "" H 3850 5000 50  0001 C CNN
+F 2 "Package_QFP:LQFP-48_7x7mm_P0.5mm" H 3850 5000 50  0001 C CNN
 F 3 "https://cdn.sparkfun.com/datasheets/Dev/Arduino/Shields/W5500_datasheet_v1.0.2_1.pdf" H 3850 5000 50  0001 C CNN
 	1    4750 4150
@@
 F 0 "JP5" H 10050 6364 50  0000 C CNN
 F 1 "Jumper" H 10050 6273 50  0000 C CNN
-F 2 "" H 10050 6100 50  0001 C CNN
+F 2 "Connector_PinSocket_2.54mm:PinSocket_1x02_P2.54mm_Vertical" H 10050 6100 50  0001 C CNN
 F 3 "~" H 10050 6100 50  0001 C CNN
 	1    10050 6100
@@
 F 0 "JP4" H 10050 6164 50  0000 C CNN
 F 1 "Jumper" H 10050 6073 50  0000 C CNN
-F 2 "" H 10050 5900 50  0001 C CNN
+F 2 "Connector_PinSocket_2.54mm:PinSocket_1x02_P2.54mm_Vertical" H 10050 5900 50  0001 C CNN
 F 3 "~" H 10050 5900 50  0001 C CNN
 	1    10050 5900
@@
 F 0 "JP2" V 4354 6477 50  0000 L CNN
 F 1 "Jumper" V 4445 6477 50  0000 L CNN
-F 2 "" H 4400 6350 50  0001 C CNN
+F 2 "Connector_PinSocket_2.54mm:PinSocket_1x02_P2.54mm_Vertical" H 4400 6350 50  0001 C CNN
 F 3 "~" H 4400 6350 50  0001 C CNN
 	1    4400 6350
@@
 F 0 "JP1" V 3854 6477 50  0000 L CNN
 F 1 "Jumper" V 3945 6477 50  0000 L CNN
-F 2 "" H 3900 6350 50  0001 C CNN
+F 2 "Connector_PinSocket_2.54mm:PinSocket_1x02_P2.54mm_Vertical" H 3900 6350 50  0001 C CNN
 F 3 "~" H 3900 6350 50  0001 C CNN
 	1    3900 6350
@@
 F 0 "JP3" V 4854 6477 50  0000 L CNN
 F 1 "Jumper" V 4945 6477 50  0000 L CNN
-F 2 "" H 4900 6350 50  0001 C CNN
+F 2 "Connector_PinSocket_2.54mm:PinSocket_1x02_P2.54mm_Vertical" H 4900 6350 50  0001 C CNN
 F 3 "~" H 4900 6350 50  0001 C CNN
 	1    4900 6350
@@
 F 0 "SW1" V 2596 5352 50  0000 R CNN
 F 1 "SW_Push" V 2505 5352 50  0000 R CNN
-F 2 "" H 2550 5600 50  0001 C CNN
+F 2 "Button_Switch_THT:SW_PUSH_6mm" H 2550 5600 50  0001 C CNN
 F 3 "~" H 2550 5600 50  0001 C CNN
 	1    2550 5400
@@
 F 0 "Y1" V 2404 4181 50  0000 L CNN
 F 1 "25MHz" V 2495 4181 50  0000 L CNN
-F 2 "" H 2450 4050 50  0001 C CNN
+F 2 "Crystal:Crystal_SMD_HC49-SD_HandSoldering" H 2450 4050 50  0001 C CNN
 F 3 "~" H 2450 4050 50  0001 C CNN
 	1    2450 4050
@@
 F 0 "FB2" H 8587 2296 50  0000 L CNN
 F 1 "BLM21" H 8587 2205 50  0000 L CNN
-F 2 "" V 8380 2250 50  0001 C CNN
+F 2 "Inductor_SMD:L_0805_2012Metric" V 8380 2250 50  0001 C CNN
 F 3 "~" H 8450 2250 50  0001 C CNN
 	1    8450 2250
@@
 F 0 "FB3" H 8587 2896 50  0000 L CNN
 F 1 "BLM21" H 8587 2805 50  0000 L CNN
-F 2 "" V 8380 2850 50  0001 C CNN
+F 2 "Inductor_SMD:L_0805_2012Metric" V 8380 2850 50  0001 C CNN
 F 3 "~" H 8450 2850 50  0001 C CNN
 	1    8450 2850
@@
 F 0 "TP2" H 8058 2268 50  0000 L CNN
 F 1 "TestPoint" H 8058 2177 50  0000 L CNN
-F 2 "" H 8200 2150 50  0001 C CNN
+F 2 "TestPoint:TestPoint_Pad_2.5x2.5mm" H 8200 2150 50  0001 C CNN
 F 3 "~" H 8200 2150 50  0001 C CNN
 	1    8000 2150
@@
 F 0 "TP1" V 7495 2922 50  0000 C CNN
 F 1 "TestPoint" V 7404 2922 50  0000 C CNN
-F 2 "" H 7500 2850 50  0001 C CNN
+F 2 "TestPoint:TestPoint_Pad_2.5x2.5mm" H 7500 2850 50  0001 C CNN
 F 3 "~" H 7500 2850 50  0001 C CNN
 	1    7300 2850
@@
 $EndComp
 $Comp
-L Connector:Barrel_Jack J2
+L Connector:Barrel_Jack_MountingPin J2
 U 1 1 6255071B
 P 10200 2450
 F 0 "J2" H 9970 2408 50  0000 R CNN
 F 1 "Barrel_Jack" H 9970 2499 50  0000 R CNN
-F 2 "" H 10250 2410 50  0001 C CNN
+F 2 "Connector_BarrelJack:BarrelJack_Horizontal" H 10250 2410 50  0001 C CNN
 F 3 "~" H 10250 2410 50  0001 C CNN
 	1    10200 2450
@@
 F 0 "D1" H 9250 6317 50  0000 C CNN
 F 1 "D" H 9250 6226 50  0000 C CNN
-F 2 "" H 9250 6100 50  0001 C CNN
+F 2 "Diode_THT:D_DO-41_SOD81_P7.62mm_Horizontal" H 9250 6100 50  0001 C CNN
 F 3 "~" H 9250 6100 50  0001 C CNN
 	1    9250 6100

Commit message: Ready to begin layout
Parts:
- J1: footprint (none) -> custom:ARJM11C7-114-BA-EW2
Changed lines of the file:
@@
 F 0 "J1" H 9928 5671 50  0000 L CNN
 F 1 "RJ45_jack_POE" H 9928 5580 50  0000 L CNN
-F 2 "" H 9600 6450 50  0001 C CNN
+F 2 "custom:ARJM11C7-114-BA-EW2" H 9600 6450 50  0001 C CNN
 F 3 "https://abracon.com/Magnetics/ARJM11.pdf" H 9600 6450 50  0001 C CNN
 	1    9600 4950
